File: PCB/TCIS.kicad_pcb (KiCad board)
At the start: 2 copper layers, 30 x 55 mm, 11 parts, among them U1 NE555P

Commit message: Updated PCB
Parts:
- C3: value 100u -> 1u
- R1: value 300K -> 330K
Connections:
- R1 pad 2: A -> B
- R2 pad 2: B -> A
- U1 pad 7: B -> A
Changed lines of the file:
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@@
 		)
 		(property "Value" "Piezo Speaker"
-			(at 0 2.46 0)
+			(at -0.5 10.295 0)
 			(unlocked yes)
 			(layer "F.Fab")
@@
 			(fill no)
 			(layer "F.SilkS")
-		)
-		(fp_text user "${REFERENCE}"
-			(at 0 5 0)
-			(unlocked yes)
-			(layer "F.Fab")
-			(effects
-				(font
-					(size 1 1)
-					(thickness 0.15)
-				)
-			)
 		)
 		(dimension
@@
 			(layers "*.Cu" "*.Mask")
 			(remove_unused_layers no)
-			(net 8 "B")
+			(net 7 "A")
 			(pinfunction "DIS")
 			(pintype "input")
@@
 			)
 		)
-		(property "Value" "100u"
+		(property "Value" "1u"
 			(at 3.75 2.42 90)
 			(layer "F.Fab")
@@
 		)
 		(property "Value" "10K"
-			(at 5.08 2.37 90)
+			(at 2.58 -2.5 90)
 			(layer "F.Fab")
 			(effects
@@
 			(layers "*.Cu" "*.Mask")
 			(remove_unused_layers no)
-			(net 8 "B")
+			(net 7 "A")
 			(pintype "passive")
 		)
@@
 		)
 		(property "Value" "100n"
-			(at 3.75 2.42 90)
+			(at 8.25 -1.5 90)
 			(layer "F.Fab")
 			(effects
@@
 			(at 5.5 5.54 90)
 			(layer "F.Fab")
+			(hide yes)
 			(effects
 				(font
@@
 			)
 			(layer "F.Fab")
-		)
-		(fp_text user "${REFERENCE}"
-			(at 2.77 1.27 0)
-			(layer "F.Fab")
-			(effects
-				(font
-					(size 1 1)
-					(thickness 0.15)
-				)
-			)
 		)
 		(pad "1" thru_hole rect
@@
 			)
 		)
-		(property "Value" "300K"
+		(property "Value" "330K"
 			(at 5.08 2.37 90)
 			(layer "F.Fab")
@@
 			(layers "*.Cu" "*.Mask")
 			(remove_unused_layers no)
-			(net 7 "A")
+			(net 8 "B")
 			(pintype "passive")
 		)
@@
 			(layer "F.Fab")
 		)
-		(fp_text user "${REFERENCE}"
-			(at -5 -1.46 0)
-			(layer "F.Fab")
-			(effects
-				(font
-					(size 1 1)
-					(thickness 0.15)
-				)
-			)
-		)
 		(pad "1" thru_hole rect
